File: src/KiCad/PN532.kicad_pcb (KiCad board)
At the start: 2 copper layers, 40 x 40 mm, 55 parts, among them J1 Bell, J2 SPOX, SW1 TAMPER, U1 PN532, U2 QR, U3 QR, Y1 27.12MHz

Commit message: update
Parts:
- removed U2, U3: QR, RevK:QR-PN532
Other:
- board text removed: "${URL}"
- board text removed: "PN532 HSU 3.3V"
- board text removed: "RFID"
